File: HW3/PIC32_breakout/PIC32_breakout.sch (EAGLE design)
At the start: 24 parts

Commit message: checked board CAM
added mounting holes and checked CAM files against Seeed. They let me add to cart so I'll assume it's fine.
Parts:
- U$2: value SWITCH_BTN_NO -> USER
- U$6: value SWITCH_BTN_NO -> RESET
Changed lines of the file:
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@@
 <part name="GND10" library="mechE433" deviceset="GND" device=""/>
 <part name="+3V6" library="mechE433" deviceset="+3V3" device=""/>
-<part name="U$6" library="mechE433" deviceset="SWITCH_BTN_NO" device=""/>
+<part name="U$6" library="mechE433" deviceset="SWITCH_BTN_NO" device="" value="RESET"/>
 <part name="GND11" library="mechE433" deviceset="GND" device=""/>
 <part name="P+1" library="mechE433" deviceset="+5V" device=""/>
@@
 <part name="C7" library="mechE433" deviceset="C-US" device="025-025X050" package3d_urn="urn:adsk.eagle:package:23629/2" value=".1uF"/>
 <part name="GND18" library="mechE433" deviceset="GND" device=""/>
-<part name="U$2" library="mechE433" deviceset="SWITCH_BTN_NO" device=""/>
+<part name="U$2" library="mechE433" deviceset="SWITCH_BTN_NO" device="" value="USER"/>
 <part name="GND19" library="mechE433" deviceset="GND" device=""/>
 <part name="+3V8" library="mechE433" deviceset="+3V3" device=""/>
